File: MIDIIn.kicad_sch (KiCad schematic)
At the start: 6 parts, among them J401 SJ2-25404B-SMT-TR, U401 TLP2361

Commit message: Replace Order_Number
Parts:
- C401, C402: footprint Capacitor_SMD:C_0603_1608Metric -> V2_Capacitor_SMD:C_0603; symbol Device:C_Small -> V2_Device:C_0603_0u1; Manufacturer (none) -> TDK; Mouser (none) -> 810-CGA3E2X7R1H104MA; Product (none) -> CGA3E2X7R1H104M080AA; Rating (none) -> 50V
- D401: footprint Diode_SMD:D_SOD-523 -> V2_Diode_SMD:D_SOD-523; Manufacturer (none) -> ROHM Semiconductor; Mouser (none) -> 755-RB501SM-30FHT2R; Product (none) -> RB501SM-30FHT2R
- J401: Manufacturer (none) -> Same Sky; Mouser (none) -> 490-SJ2-25404BSMT-TR; Product (none) -> SJ2-25404B-SMT-TR
- R401: footprint Resistor_SMD:R_0603_1608Metric -> V2_Resistor_SMD:R_0603; symbol Device:R_Small -> V2_Device:R_0603_220R; Manufacturer (none) -> Vishay; Mouser (none) -> 71-CRCW0603220RFKEAH; Product (none) -> CRCW0603220RFKEAHP; Rating (none) -> 330mW
- U401: footprint Package_SO:SO-5-6_4.55x3.7mm_P1.27mm -> V2_Package_SO:SO-5-6_4.55x3.7mm_P1.27mm; Manufacturer (none) -> Toshiba; Mouser (none) -> 757-TLP2361TPRE; Product (none) -> TLP2361(TPR,E

Commit message: Update Library
Parts:
- C401, C402: symbol V2_Device:C_0603_0u1 -> V2_Capacitor:0603_0u1
- R401: symbol V2_Device:R_0603_220R -> V2_Resistor:0603_220R

Commit message: Replace diode
Parts:
- D401: value RB501SM -> PMEG2010EPK; footprint V2_Diode_SMD:D_SOD-523 -> V2_Diode_SMD:D_SOD-1608; symbol V2_Diode:RB501SM -> V2_Diode:PMEG2010EPK; Manufacturer ROHM Semiconductor -> Nexperia; Mouser 755-RB501SM-30FHT2R -> 771-PMEG2010EPK; Product RB501SM-30FHT2R -> PMEG2010EPK; Rating (none) -> 20V
Other:
- title: MIDI In -> V2 control
Changed lines of the file:
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@@
 (kicad_sch
-	(version 20250114)
+	(version 20260306)
 	(generator "eeschema")
-	(generator_version "9.0")
+	(generator_version "10.0")
 	(paper "A4")
 	(title_block
-		(title "MIDI In")
-		(date "2026-02-11")
-		(rev "2026-02-11")
+		(title "V2 control")
+		(date "2026-03-30")
+		(rev "2026-03-30")
 	)

Commit message: Good Bye Imperial
Parts:
- C401, C402: footprint V2_Capacitor_SMD:C_0603 -> V2_Capacitor_SMD:C_1608; symbol V2_Capacitor:0603_0u1 -> V2_Capacitor:1608_0u1
- R401: footprint V2_Resistor_SMD:R_0603 -> V2_Resistor_SMD:R_1608; symbol V2_Resistor:0603_220R -> V2_Resistor:1608_220R
